File: OrigJrBoard/JrBoard/JrBoard.sch (KiCad schematic (older format))
At the start: 47 parts, among them J1 DB9_Male, J2 AudioJack2_Ground, J3 DB9_Male, J5 Conn_02x12_Counter_Clockwise, Q4 2N3904

Commit message: Continued schematic
Parts:
- removed A1: 6532, symbol Interface_MOS:6532
- removed CR3, CR4: D, symbol Device:D
- removed R31: R, symbol Device:R
- added A1: 6532, symbol Atari2600Jr:6532
- added A2: 6507, Package_DIP:DIP-28_W15.24mm, symbol Atari2600Jr:6507
- added A3: UM6526P1, symbol Atari2600Jr:UM6526P1
- added unit 2 of A4
- added unit 5 of A4
- added unit 4 of A4
- added unit 6 of A4
- added unit 1 of A4
- added A5: LM3086N, symbol Atari2600Jr:LM3086N
- added C10, C11, C13, C14, C15, C16, C17, C18, C19, C22, C30, C31, C32, C33, C34, C35, C39, C40, C41, C43, C46, C47, C48, C49, C5, C50, C51, C52, C54, C55, C6, C7, C8, C9: C, symbol Device:C
- added C20, C27: CP, symbol Device:CP
- added CR2, CR3, CR4, CR5: 1N4148, Diode_THT:D_DO-35_SOD27_P7.62mm_Horizontal, symbol Diode:1N4148
- added J4: RF_Out, symbol Connector:Conn_Coaxial
- added L5, L9: L, symbol Device:L
- added L6: LTRIM, symbol Device:LTRIM
- added Q1, Q2, Q3: 2N3906, Package_TO_SOT_THT:TO-92_Inline, symbol Transistor_BJT:2N3906
- added Q5: 2N3904, Package_TO_SOT_THT:TO-92_Inline, symbol Transistor_BJT:2N3904
- added R1, R10, R11, R12, R15, R17, R18, R19, R2, R20, R21, R25, R26, R27, R28, R3, R32, R36, R37, R38, R39, R40, R41, R42, R43, R44, R45, R47, R48, R49, R5, R51, R52, R53, R55, R56, R6, R8: R, symbol Device:R
- added R50, R54: DNF, symbol Device:R
- added R9: R_POT_Small, symbol Device:R_POT_Small
- added T1: TV_Trans, Atari2600Jr:Atari_TV_Trans, symbol Atari2600Jr:TV_Trans
- added TP1: 5V, symbol Connector:TestPoint
- added TP2: A1_RES, symbol Connector:TestPoint
- added TP3: 3.54MHz, symbol Connector:TestPoint
- added TP4: A2_RES, symbol Connector:TestPoint
- added TP5: A/V, symbol Connector:TestPoint
- added TP6: 4.43MHz, symbol Connector:TestPoint
- added TP7: Audio, symbol Connector:TestPoint
- added U4: 4050, symbol 4xxx_IEEE:4050
- added W2: DNF, symbol Jumper:Jumper_2_Open
- added Y1: 3.546894MHz, symbol Device:Crystal
- added Y2: 4.433618MHz, symbol Device:Crystal
- J1: value DB9_Male -> Joy left
- J2: value AudioJack2_Ground -> DC In
- J3: value DB9_Male -> Joy right
- J5: value Conn_02x12_Counter_Clockwise -> Cartridge Connector
- S1: value SW_SPDT -> CH3/4
- renumbered R41 to R31
Connections:
- net labels added: +5V, +5VA, A0, A1, A10, A11, A12, A1_R, A2, A2_R, A3, A4, A5, A6, A7, A8, A9, AUD, COL, CSYNC, D7, I0, I1, I2, I3, I4, I5, LUM0, LUM1, LUM2, OSC, PA0, PA1, PA2, PA3, PA4, PA5, PA6, PA7, PAL-S, RDY, o0, o2
- wire segments 82 -> 479
Other:
- moved on the sheet: A4G, C12, C28, C29, C4, C53, J1, J3, J5, L11, L2, L3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

Commit message: Continued schematic
Parts:
- added C1, C23, C24, C25, C3: 1n, symbol Device:C
- added J6: SEL / RES, symbol Connector_Generic:Conn_01x06
- added S2: DIFF_L, symbol Switch:SW_SPDT
- added S3: DIFF_R, symbol Switch:SW_SPDT
- added S5: COLOR_SW, symbol Switch:SW_SPDT
- added W1, W3: DNF, symbol Jumper:Jumper_2_Open
- C10, C15, C16, C17, C18, C34, C4, C7, C8, C9: value C -> 1n
- C11, C19: value C -> 470p
- C12, C2, C21, C22, C28, C36, C38, C41, C43, C47, C49: value C -> 100n
- C13, C14, C5, C6: value C -> 68n
- C20, C27, C29, C37: value CP -> 4u7
- C26: value CP -> 2m2
- C30: value C -> 39p
- C31: value C -> DNF
- C32: value C -> 18p
- C33: value C -> 100p
- C35: value C -> 68p
- C39: value C -> 10n
- C40: value C -> 10p
- C46: value C -> 56p
- C48, C53, C54: value C -> 820p
- C50: value C -> 47n
- C51, C55: value C -> 22p
- C52: value C -> 47p
- DS1: value LED -> LED RED
- L1, L11, L2, L4, L5, L7: value L -> 1u
- L3: value L -> 15u
- L6: value LTRIM -> 0..1u
- L8: value LTRIM -> 0..4u
- L9: value L -> 1u5
- R1, R2, R5, R6: value R -> 1K8
- R10, R26, R3, R8: value R -> 220
- R11: value R -> 240
- R12, R18, R19, R27: value R -> 100
- R14: value R -> 3K3
- R15, R4, R7: value R -> 10K
- R16: value R -> 2K7
- R17: value R -> 330
- R20, R24: value R -> 1K
- R21: value R -> 1K5
- R22: value R -> 4K7
- R23: value R -> 91
- R25: value R -> 2K2
- R28: value R -> 1M
- R9: value R_POT_Small -> 500K
- S4: value SW_SPDT -> POWER_SW
- renumbered U4 to A4
Connections:
- net D7: now also A1.26 (D7), A3.34 (D7), J5.17 (Pin_17)
- net GND: now also A3.22 (CS2), C1.2, C23.2, C24.2, C25.2, C3.2, J6.6 (Pin_6), S2.1 (A), S2.2 (B), S3.1 (A), S3.2 (B), S5.1 (A), S5.2 (B)
- net OSC: now also W1.1 (A)
- net D6: now reaches A2.19 (D6)
- net D6: now also A1.27 (D6), A3.33 (D6), J5.16 (Pin_16)
- net D5: now reaches A2.20 (D5)
- net D5: now also A1.28 (D5), A3.19 (D5), J5.15 (Pin_15)
- net D4: now reaches A2.21 (D4)
- net D4: now also A1.29 (D4), A3.18 (D4), J5.14 (Pin_14)
- net D3: now reaches A2.22 (D3)
- net D3: now also A1.30 (D3), A3.17 (D3), J5.13 (Pin_13)
- net D2: now reaches A2.23 (D2)
- net D2: now also A1.31 (D2), A3.16 (D2), J5.11 (Pin_11)
- net D1: now reaches A2.24 (D1)
- net D1: now also A1.32 (D1), A3.15 (D1), J5.10 (Pin_10)
- net D0: now reaches A2.25 (D0)
- net D0: now also A1.33 (D0), A3.14 (D0), J5.9 (Pin_9)
- net RW: now reaches A2.26 (R/W)
- net RW: now also A1.35 (R/W), A3.25 (R/W)
- net at A3.8 (PAL-I), R47.1: now also W1.2 (B), W3.1 (A)
- net PB7: now reaches A1.16 (PB7)
- net PB7: now also C3.1, S3.3 (C)
- net PB6: now reaches A1.17 (PB6)
- net PB6: now also C1.1, S2.3 (C)
- net PB3: now reaches A1.21 (PB3)
- net PB3: now also C23.1, S5.3 (C)
- net PB1: now reaches A1.23 (PB1)
- net PB1: now also C24.1, J6.2 (Pin_2)
- net PB0: now reaches A1.24 (PB0)
- net PB0: now also C25.1, J6.4 (Pin_4)
- net at R14.2: now also A4.7, W3.2 (B); no longer A4.6
- net at R50.2: now also A4.6; no longer A4.7
Other:
- moved on the sheet: C11, C19, C2, C21, C36, C43, L4, R4, R44, R7

Commit message: finished schematic
Parts:
- A1, A3: footprint (none) -> Package_DIP:DIP-40_W15.24mm
- A4: footprint (none) -> Package_DIP:DIP-16_W7.62mm
- A5: footprint (none) -> Package_DIP:DIP-14_W7.62mm
- DS1: footprint (none) -> LED_THT:LED_D5.0mm_Clear
- Q1, Q2, Q3, Q4, Q5: footprint Package_TO_SOT_THT:TO-92_Inline -> Package_TO_SOT_THT:TO-92
- R29, R34, R46: value R -> 1K
- R30, R33, R35, R41: value R -> 3K3
- R31, R45, R51, R53: value R -> 10K
- R32, R47: value R -> 100
- R36, R39: value R -> 4K7
- R37: value R -> 470
- R38: value R -> 12K
- R40: value R -> 100K
- R42, R44, R55: value R -> 6K8
- R43: value R -> 9K1
- R48: value R -> 18K
- R49: value R -> 20K
- R52: value R -> 39K
- R56: value R -> 1K8
- R57: value R -> 750
- TP1, TP2, TP3, TP4, TP5, TP6, TP7: footprint (none) -> TestPoint:TestPoint_Plated_Hole_D2.0mm
- VR1: footprint (none) -> Package_TO_SOT_THT:TO-220-3_Horizontal_TabDown

Commit message: Started PCB
Parts:
- C1, C10, C11, C12, C15, C16, C17, C18, C19, C2, C21, C22, C23, C24, C25, C28, C3, C33, C34, C35, C36, C38, C39, C4, C40, C41, C43, C46, C47, C49, C50, C51, C52, C55, C7, C8, C9: footprint (none) -> Atari2600Jr:C_leg_small
- C13, C14, C5, C6: footprint (none) -> Atari2600Jr:C_oval_big
- C20, C27, C29, C37: footprint (none) -> Atari2600Jr:CP_small
- C26: footprint (none) -> Atari2600Jr:CP_big
- C30, C31: footprint (none) -> Atari2600Jr:C_oval_small
- C32: footprint (none) -> Atari2600Jr:C_4hole
- C48, C53, C54: footprint (none) -> Atari2600Jr:C_leg_big
- CR2, CR3, CR4, CR5: footprint Diode_THT:D_DO-35_SOD27_P7.62mm_Horizontal -> Atari2600Jr:Diode
- J1, J3: footprint (none) -> Atari2600Jr:Joystick_conn
- J2: footprint (none) -> Atari2600Jr:DC_IN
- J4: footprint (none) -> Atari2600Jr:RF_Out
- J5: footprint (none) -> Atari2600Jr:Cartridge
- J6: footprint (none) -> Atari2600Jr:Button_conn
- L1, L11, L2, L4, L5, L7: footprint (none) -> Atari2600Jr:L_small
- L3, L9: footprint (none) -> Atari2600Jr:L_big
- L6: footprint (none) -> Atari2600Jr:L_var_2pin
- L8: footprint (none) -> Atari2600Jr:L_var_5pin
- R1, R10, R11, R12, R14, R15, R16, R17, R18, R19, R2, R20, R21, R22, R23, R24, R25, R26, R27, R28, R29, R3, R30, R31, R32, R33, R34, R35, R36, R37, R38, R39, R4, R40, R41, R42, R43, R44, R45, R46, R47, R48, R49, R5, R50, R51, R52, R53, R54, R55, R56, R57, R6, R7, R8: footprint (none) -> Atari2600Jr:R0.5Inch
- R9: footprint (none) -> Atari2600Jr:R_Var
- S1, S2, S3: footprint (none) -> Atari2600Jr:Switch_rear
- S4, S5: footprint (none) -> Atari2600Jr:Switch_top
- W1, W2, W3: footprint (none) -> Atari2600Jr:Wire
- Y1, Y2: footprint (none) -> Crystal:Crystal_HC18-U_Vertical

Commit message: PCB work
Parts:
- removed unit 2 of A4
- removed unit 3 of A4
- removed unit 5 of A4
- removed unit 4 of A4
- removed unit 6 of A4
- removed unit 1 of A4
- added unit 2 of A4
- added unit 3 of A4
- added unit 1 of A4
- added unit 4 of A4
- added unit 5 of A4
- added unit 6 of A4
Connections:
- net A2_R: now also A4.4
- net CSYNC: now also A4.11
- net LUM0: now also A4.3
- net LUM1: now also A4.9
- net LUM2: now also A4.14
- net at R14.2, W3.2 (B): now also A4.7
- net at R28.1, R40.2: now also A4.5
- net at R50.2: now also A4.6
- net at R51.2: now also A4.12
- net at R49.2: now also A4.10
- net at R53.2, R54.2: now also A4.15
- net at R52.2: now also A4.2
- no-connect marks 0 -> 7

Commit message: PCB work
Connections:
- net GND: now also S5.3 (C); no longer S5.1 (A)
- net PB3: now also S5.1 (A); no longer S5.3 (C)
Other:
- moved on the sheet: C23
Changed lines of the file:
@@
 EESchema Schematic File Version 4
+LIBS:JrBoard-cache
 EELAYER 30 0
 EELAYER END
@@
 $EndComp
 $Comp
-L Device:C C23
-U 1 1 635C99AC
-P 9950 2350
-F 0 "C23" H 10065 2396 50  0000 L CNN
-F 1 "1n" H 10065 2305 50  0000 L CNN
-F 2 "Atari2600Jr:C_leg_small" H 9988 2200 50  0001 C CNN
-F 3 "~" H 9950 2350 50  0001 C CNN
-	1    9950 2350
-	1    0    0    -1
-$EndComp
-Wire Wire Line
-	10350 2250 10250 2250
-Wire Wire Line
-	10250 2250 10250 2200
-Wire Wire Line
-	10250 2200 9950 2200
-Wire Wire Line
-	10350 2450 10250 2450
-Wire Wire Line
-	10250 2450 10250 2500
-Wire Wire Line
-	10250 2500 9950 2500
-Wire Wire Line
-	10350 2450 10350 2650
-Wire Wire Line
-	10350 2650 10750 2650
-Wire Wire Line
-	10750 2650 10750 2350
-Connection ~ 10350 2450
-$Comp
 L power:GND #PWR0182
 U 1 1 636BF123
-P 9950 2500
-F 0 "#PWR0182" H 9950 2250 50  0001 C CNN
-F 1 "GND" H 9955 2327 50  0000 C CNN
-F 2 "" H 9950 2500 50  0001 C CNN
-F 3 "" H 9950 2500 50  0001 C CNN
-	1    9950 2500
+P 11100 2350
+F 0 "#PWR0182" H 11100 2100 50  0001 C CNN
+F 1 "GND" H 11105 2177 50  0000 C CNN
+F 2 "" H 11100 2350 50  0001 C CNN
+F 3 "" H 11100 2350 50  0001 C CNN
+	1    11100 2350
 	1    0    0    -1
 $EndComp
-Connection ~ 9950 2500
 Entry Wire Line
 	5550 7700 5450 7600
@@
 Entry Wire Line
 	11550 2050 11450 1950
-Wire Wire Line
-	11450 1950 10250 1950
-Wire Wire Line
-	10250 1950 10250 2200
-Connection ~ 10250 2200
 Text Label 11300 1950 0    50   ~ 0
 PB3
@@
 Wire Wire Line
 	5500 2400 5750 2400
-Wire Bus Line
-	9900 9650 11550 9650
-Wire Bus Line
-	3150 7150 3150 9650
-Wire Bus Line
-	9900 6600 9900 9650
-Wire Bus Line
-	2100 6950 2100 9650
-Wire Bus Line
-	8050 6850 8050 9650
-Wire Bus Line
-	6700 6850 6700 9650
-Wire Bus Line
-	5550 6600 5550 9650
-Wire Bus Line
-	3850 6600 3850 9650
-Wire Bus Line
-	11550 1750 11550 9650
 Connection ~ 5500 2400
 $Comp
@@
 $EndComp
 Connection ~ 1000 1500
+Wire Wire Line
+	10150 1950 10150 2450
+Wire Wire Line
+	10150 2450 10350 2450
+Wire Wire Line
+	10150 1950 11100 1950
+Wire Wire Line
+	10350 2250 10350 2150
+Wire Wire Line
+	10350 2150 10900 2150
+Wire Wire Line
+	10900 2150 10900 2350
+Wire Wire Line
+	10900 2350 10750 2350
+$Comp
+L Device:C C23
+U 1 1 635C99AC
+P 11100 2200
+F 0 "C23" H 11215 2246 50  0000 L CNN
+F 1 "1n" H 11215 2155 50  0000 L CNN
+F 2 "Atari2600Jr:C_leg_small" H 11138 2050 50  0001 C CNN
+F 3 "~" H 11100 2200 50  0001 C CNN
+	1    11100 2200
+	1    0    0    -1
+$EndComp
+Wire Wire Line
+	11100 2050 11100 1950
+Connection ~ 11100 1950
+Wire Wire Line
+	11100 1950 11450 1950
+Wire Wire Line
+	10900 2350 11100 2350
+Wire Bus Line
+	9900 9650 11550 9650
+Wire Bus Line
+	3150 7150 3150 9650
+Wire Bus Line
+	9900 6600 9900 9650
+Wire Bus Line
+	2100 6950 2100 9650
+Wire Bus Line
+	8050 6850 8050 9650
+Wire Bus Line
+	6700 6850 6700 9650
+Wire Bus Line
+	5550 6600 5550 9650
+Wire Bus Line
+	3850 6600 3850 9650
+Wire Bus Line
+	11550 1750 11550 9650
+Connection ~ 10900 2350
+Connection ~ 11100 2350
 $EndSCHEMATC

Commit message: PCB top mostly done
Parts:
- CR2: footprint Atari2600Jr:Diode -> Atari2600Jr:Diode_short
- Q1, Q2, Q3, Q4, Q5: footprint Package_TO_SOT_THT:TO-92 -> Atari2600Jr:TR_TO92
- R15, R16, R17, R18, R20, R21: footprint Atari2600Jr:R0.5Inch -> Atari2600Jr:R_small
- TP1, TP2, TP3, TP4, TP5, TP6, TP7: footprint TestPoint:TestPoint_Plated_Hole_D2.0mm -> TestPoint:TestPoint_Pad_D1.5mm
Changed lines of the file:
@@
 EESchema Schematic File Version 4
-LIBS:JrBoard-cache
 EELAYER 30 0
 EELAYER END
@@
 F 0 "R16" H 15300 4850 50  0000 C CNN
 F 1 "2K7" H 15300 4950 50  0000 C CNN
-F 2 "Atari2600Jr:R0.5Inch" V 15380 4900 50  0001 C CNN
+F 2 "Atari2600Jr:R_small" V 15380 4900 50  0001 C CNN
 F 3 "~" H 15450 4900 50  0001 C CNN
 	1    15450 4900
@@
 F 0 "Q4" V 15635 9300 50  0000 C CNN
 F 1 "2N3904" V 15726 9300 50  0000 C CNN
-F 2 "Package_TO_SOT_THT:TO-92" H 15600 9225 50  0001 L CIN
+F 2 "Atari2600Jr:TR_TO92" H 15600 9225 50  0001 L CIN
 F 3 "https://www.fairchildsemi.com/datasheets/2N/2N3904.pdf" H 15400 9300 50  0001 L CNN
 	1    15400 9300
@@
 F 0 "R18" H 14070 4946 50  0000 L CNN
 F 1 "100" H 14070 4855 50  0000 L CNN
-F 2 "Atari2600Jr:R0.5Inch" V 13930 4900 50  0001 C CNN
+F 2 "Atari2600Jr:R_small" V 13930 4900 50  0001 C CNN
 F 3 "~" H 14000 4900 50  0001 C CNN
 	1    14000 4900
@@
 F 0 "Q2" H 2141 3454 50  0000 L CNN
 F 1 "2N3906" H 2141 3545 50  0000 L CNN
-F 2 "Package_TO_SOT_THT:TO-92" H 2150 3425 50  0001 L CIN
+F 2 "Atari2600Jr:TR_TO92" H 2150 3425 50  0001 L CIN
 F 3 "https://www.fairchildsemi.com/datasheets/2N/2N3906.pdf" H 1950 3500 50  0001 L CNN
 	1    1950 3500
@@
 F 0 "Q1" H 1441 3454 50  0000 L CNN
 F 1 "2N3906" H 1441 3545 50  0000 L CNN
-F 2 "Package_TO_SOT_THT:TO-92" H 1450 3425 50  0001 L CIN
+F 2 "Atari2600Jr:TR_TO92" H 1450 3425 50  0001 L CIN
 F 3 "https://www.fairchildsemi.com/datasheets/2N/2N3906.pdf" H 1250 3500 50  0001 L CNN
 	1    1250 3500
@@
 F 0 "Q5" H 3990 3496 50  0000 L CNN
 F 1 "2N3904" H 3990 3405 50  0000 L CNN
-F 2 "Package_TO_SOT_THT:TO-92" H 4000 3375 50  0001 L CIN
+F 2 "Atari2600Jr:TR_TO92" H 4000 3375 50  0001 L CIN
 F 3 "https://www.fairchildsemi.com/datasheets/2N/2N3904.pdf" H 3800 3450 50  0001 L CNN
 	1    3800 3450
@@
 F 0 "Q3" H 13640 4546 50  0000 L CNN
 F 1 "2N3906" H 13640 4455 50  0000 L CNN
-F 2 "Package_TO_SOT_THT:TO-92" H 13650 4425 50  0001 L CIN
+F 2 "Atari2600Jr:TR_TO92" H 13650 4425 50  0001 L CIN
 F 3 "https://www.fairchildsemi.com/datasheets/2N/2N3906.pdf" H 13450 4500 50  0001 L CNN
 	1    13450 4500
@@
 F 0 "R21" H 12320 5496 50  0000 L CNN
 F 1 "1K5" H 12320 5405 50  0000 L CNN
-F 2 "Atari2600Jr:R0.5Inch" V 12180 5450 50  0001 C CNN
+F 2 "Atari2600Jr:R_small" V 12180 5450 50  0001 C CNN
 F 3 "~" H 12250 5450 50  0001 C CNN
 	1    12250 5450
@@
 F 0 "R20" H 12320 5996 50  0000 L CNN
 F 1 "1K" H 12320 5905 50  0000 L CNN
-F 2 "Atari2600Jr:R0.5Inch" V 12180 5950 50  0001 C CNN
+F 2 "Atari2600Jr:R_small" V 12180 5950 50  0001 C CNN
 F 3 "~" H 12250 5950 50  0001 C CNN
 	1    12250 5950
@@
 F 0 "R15" H 12420 4496 50  0000 L CNN
 F 1 "10K" H 12420 4405 50  0000 L CNN
-F 2 "Atari2600Jr:R0.5Inch" V 12280 4450 50  0001 C CNN
+F 2 "Atari2600Jr:R_small" V 12280 4450 50  0001 C CNN
 F 3 "~" H 12350 4450 50  0001 C CNN
 	1    12350 4450
@@
 F 0 "CR2" V 11796 5621 50  0000 R CNN
 F 1 "1N4148" V 11705 5621 50  0000 R CNN
-F 2 "Atari2600Jr:Diode" H 11750 5525 50  0001 C CNN
+F 2 "Atari2600Jr:Diode_short" H 11750 5525 50  0001 C CNN
 F 3 "https://assets.nexperia.com/documents/data-sheet/1N4148_1N4448.pdf" H 11750 5700 50  0001 C CNN
 	1    11750 5700
@@
 F 0 "R17" H 15820 5696 50  0000 L CNN
 F 1 "330" H 15820 5605 50  0000 L CNN
-F 2 "Atari2600Jr:R0.5Inch" V 15680 5650 50  0001 C CNN
+F 2 "Atari2600Jr:R_small" V 15680 5650 50  0001 C CNN
 F 3 "~" H 15750 5650 50  0001 C CNN
 	1    15750 5650
@@
 F 0 "TP7" H 14658 7768 50  0000 L CNN
 F 1 "Audio" H 14658 7677 50  0000 L CNN
-F 2 "TestPoint:TestPoint_Plated_Hole_D2.0mm" H 14800 7650 50  0001 C CNN
+F 2 "TestPoint:TestPoint_Pad_D1.5mm" H 14800 7650 50  0001 C CNN
 F 3 "~" H 14800 7650 50  0001 C CNN
 	1    14600 7650
@@
 F 0 "TP5" H 15008 6318 50  0000 L CNN
 F 1 "A/V" H 15008 6227 50  0000 L CNN
-F 2 "TestPoint:TestPoint_Plated_Hole_D2.0mm" H 15150 6200 50  0001 C CNN
+F 2 "TestPoint:TestPoint_Pad_D1.5mm" H 15150 6200 50  0001 C CNN
 F 3 "~" H 15150 6200 50  0001 C CNN
 	1    14950 6200
@@
 F 0 "TP4" H 5908 7218 50  0000 L CNN
 F 1 "A2_RES" H 5908 7127 50  0000 L CNN
-F 2 "TestPoint:TestPoint_Plated_Hole_D2.0mm" H 6050 7100 50  0001 C CNN
+F 2 "TestPoint:TestPoint_Pad_D1.5mm" H 6050 7100 50  0001 C CNN
 F 3 "~" H 6050 7100 50  0001 C CNN
 	1    5850 7100
@@
 F 0 "TP1" H 4158 1018 50  0000 L CNN
 F 1 "5V" H 4158 927 50  0000 L CNN
-F 2 "TestPoint:TestPoint_Plated_Hole_D2.0mm" H 4300 900 50  0001 C CNN
+F 2 "TestPoint:TestPoint_Pad_D1.5mm" H 4300 900 50  0001 C CNN
 F 3 "~" H 4300 900 50  0001 C CNN
 	1    4100 900
@@
 F 0 "TP6" V 4154 3388 50  0000 L CNN
 F 1 "4.43MHz" V 4245 3388 50  0000 L CNN
-F 2 "TestPoint:TestPoint_Plated_Hole_D2.0mm" H 4400 3200 50  0001 C CNN
+F 2 "TestPoint:TestPoint_Pad_D1.5mm" H 4400 3200 50  0001 C CNN
 F 3 "~" H 4400 3200 50  0001 C CNN
 	1    4200 3200
@@
 F 0 "TP3" H 758 3418 50  0000 L CNN
 F 1 "3.54MHz" H 758 3327 50  0000 L CNN
-F 2 "TestPoint:TestPoint_Plated_Hole_D2.0mm" H 900 3300 50  0001 C CNN
+F 2 "TestPoint:TestPoint_Pad_D1.5mm" H 900 3300 50  0001 C CNN
 F 3 "~" H 900 3300 50  0001 C CNN
 	1    700  3300
@@
 Wire Wire Line
 	5750 6100 6250 6100
-$Comp
-L Connector:TestPoint TP2
-U 1 1 61E63A0B
-P 5350 5450
-F 0 "TP2" H 5408 5568 50  0000 L CNN
-F 1 "A1_RES" H 5408 5477 50  0000 L CNN
-F 2 "TestPoint:TestPoint_Plated_Hole_D2.0mm" H 5550 5450 50  0001 C CNN
-F 3 "~" H 5550 5450 50  0001 C CNN
-	1    5350 5450
-	1    0    0    -1
-$EndComp
 Wire Wire Line
 	5350 5450 5350 5550
@@
 Wire Wire Line
 	10900 2350 11100 2350
+Connection ~ 10900 2350
+Connection ~ 11100 2350
 Wire Bus Line
 	9900 9650 11550 9650
@@
 Wire Bus Line
 	11550 1750 11550 9650
-Connection ~ 10900 2350
-Connection ~ 11100 2350
+$Comp
+L Connector:TestPoint TP2
+U 1 1 61E63A0B
+P 5350 5450
+F 0 "TP2" H 5408 5568 50  0000 L CNN
+F 1 "A1_RES" H 5408 5477 50  0000 L CNN
+F 2 "TestPoint:TestPoint_Pad_D1.5mm" H 5550 5450 50  0001 C CNN
+F 3 "~" H 5550 5450 50  0001 C CNN
+	1    5350 5450
+	1    0    0    -1
+$EndComp
 $EndSCHEMATC
