File: OrigJrBoard/JrBoard/JrBoard.sch (KiCad schematic (older format))
At the start: 158 parts, among them J1 Joy left, J2 DC In, J3 Joy right, J4 RF_Out, J5 Cartridge Connector, J6 SEL / RES, Q1 2N3906, Q2 2N3906, Q3 2N3906, Q4 2N3904, Q5 2N3904, T1 TV_Trans, Y1 3.546894MHz, Y2 4.433618MHz

Commit message: Finished PCB
Parts:
- TP1, TP2, TP3, TP4, TP5, TP6, TP7: footprint TestPoint:TestPoint_Pad_D1.5mm -> TestPoint:TestPoint_THTPad_D2.0mm_Drill1.0mm
Connections:
- net GND: no longer R16.2
- net at C4.1, S1.2 (B): now also R16.2
Other:
- moved on the sheet: C4, R16, S1
Changed lines of the file:
@@
 EESchema Schematic File Version 4
+LIBS:JrBoard-cache
 EELAYER 30 0
 EELAYER END
@@
 L Switch:SW_SPDT S1
 U 1 1 5FD13744
-P 15450 4450
-F 0 "S1" H 15450 4125 50  0000 C CNN
-F 1 "CH3/4" H 15450 4216 50  0000 C CNN
-F 2 "Atari2600Jr:Switch_rear" H 15450 4450 50  0001 C CNN
-F 3 "~" H 15450 4450 50  0001 C CNN
-	1    15450 4450
+P 15450 4350
+F 0 "S1" H 15450 4025 50  0000 C CNN
+F 1 "CH3/4" H 15450 4116 50  0000 C CNN
+F 2 "Atari2600Jr:Switch_rear" H 15450 4350 50  0001 C CNN
+F 3 "~" H 15450 4350 50  0001 C CNN
+	1    15450 4350
 	-1   0    0    1
 $EndComp
@@
 L power:GND #PWR0113
 U 1 1 5FD14BED
-P 15250 4700
-F 0 "#PWR0113" H 15250 4450 50  0001 C CNN
-F 1 "GND" H 15255 4527 50  0000 C CNN
-F 2 "" H 15250 4700 50  0001 C CNN
-F 3 "" H 15250 4700 50  0001 C CNN
-	1    15250 4700
+P 15250 4600
+F 0 "#PWR0113" H 15250 4350 50  0001 C CNN
+F 1 "GND" H 15255 4427 50  0000 C CNN
+F 2 "" H 15250 4600 50  0001 C CNN
+F 3 "" H 15250 4600 50  0001 C CNN
+	1    15250 4600
 	1    0    0    -1
 $EndComp
-Wire Wire Line
-	15250 4700 15250 4650
 $Comp
 L Device:C C4
 U 1 1 5FD156F9
-P 15650 4600
-F 0 "C4" H 15765 4646 50  0000 L CNN
-F 1 "1n" H 15765 4555 50  0000 L CNN
-F 2 "Atari2600Jr:C_leg_small" H 15688 4450 50  0001 C CNN
-F 3 "~" H 15650 4600 50  0001 C CNN
-	1    15650 4600
+P 15650 4500
+F 0 "C4" H 15765 4546 50  0000 L CNN
+F 1 "1n" H 15765 4455 50  0000 L CNN
+F 2 "Atari2600Jr:C_leg_small" H 15688 4350 50  0001 C CNN
+F 3 "~" H 15650 4500 50  0001 C CNN
+	1    15650 4500
 	1    0    0    -1
 $EndComp
-Wire Wire Line
-	15650 4750 15450 4750
-Wire Wire Line
-	15450 4750 15450 4650
-Wire Wire Line
-	15450 4650 15250 4650
-Connection ~ 15250 4650
-Wire Wire Line
-	15250 4650 15250 4550
 $Comp
 L Device:R R16
 U 1 1 5FD16867
-P 15450 4900
-F 0 "R16" H 15300 4850 50  0000 C CNN
-F 1 "2K7" H 15300 4950 50  0000 C CNN
-F 2 "Atari2600Jr:R_small" V 15380 4900 50  0001 C CNN
-F 3 "~" H 15450 4900 50  0001 C CNN
-	1    15450 4900
+P 15650 4900
+F 0 "R16" H 15500 4850 50  0000 C CNN
+F 1 "2K7" H 15500 4950 50  0000 C CNN
+F 2 "Atari2600Jr:R_small" V 15580 4900 50  0001 C CNN
+F 3 "~" H 15650 4900 50  0001 C CNN
+	1    15650 4900
 	-1   0    0    1
 $EndComp
@@
 L power:+5V #PWR0152
 U 1 1 60401A39
-P 15250 4350
-F 0 "#PWR0152" H 15250 4200 50  0001 C CNN
-F 1 "+5V" V 15265 4478 50  0000 L CNN
-F 2 "" H 15250 4350 50  0001 C CNN
-F 3 "" H 15250 4350 50  0001 C CNN
-	1    15250 4350
+P 15250 4250
+F 0 "#PWR0152" H 15250 4100 50  0001 C CNN
+F 1 "+5V" V 15265 4378 50  0000 L CNN
+F 2 "" H 15250 4250 50  0001 C CNN
+F 3 "" H 15250 4250 50  0001 C CNN
+	1    15250 4250
 	0    -1   -1   0
 $EndComp
@@
 	13550 5600 13450 5600
 Connection ~ 13550 5400
-Connection ~ 15450 4750
-Wire Wire Line
-	15450 5050 14750 5050
 Wire Wire Line
 	14750 5050 14750 4200
@@
 F 0 "TP7" H 14658 7768 50  0000 L CNN
 F 1 "Audio" H 14658 7677 50  0000 L CNN
-F 2 "TestPoint:TestPoint_Pad_D1.5mm" H 14800 7650 50  0001 C CNN
+F 2 "TestPoint:TestPoint_THTPad_D2.0mm_Drill1.0mm" H 14800 7650 50  0001 C CNN
 F 3 "~" H 14800 7650 50  0001 C CNN
 	1    14600 7650
@@
 F 0 "TP5" H 15008 6318 50  0000 L CNN
 F 1 "A/V" H 15008 6227 50  0000 L CNN
-F 2 "TestPoint:TestPoint_Pad_D1.5mm" H 15150 6200 50  0001 C CNN
+F 2 "TestPoint:TestPoint_THTPad_D2.0mm_Drill1.0mm" H 15150 6200 50  0001 C CNN
 F 3 "~" H 15150 6200 50  0001 C CNN
 	1    14950 6200
@@
 F 0 "TP4" H 5908 7218 50  0000 L CNN
 F 1 "A2_RES" H 5908 7127 50  0000 L CNN
-F 2 "TestPoint:TestPoint_Pad_D1.5mm" H 6050 7100 50  0001 C CNN
+F 2 "TestPoint:TestPoint_THTPad_D2.0mm_Drill1.0mm" H 6050 7100 50  0001 C CNN
 F 3 "~" H 6050 7100 50  0001 C CNN
 	1    5850 7100
@@
 F 0 "TP1" H 4158 1018 50  0000 L CNN
 F 1 "5V" H 4158 927 50  0000 L CNN
-F 2 "TestPoint:TestPoint_Pad_D1.5mm" H 4300 900 50  0001 C CNN
+F 2 "TestPoint:TestPoint_THTPad_D2.0mm_Drill1.0mm" H 4300 900 50  0001 C CNN
 F 3 "~" H 4300 900 50  0001 C CNN
 	1    4100 900
@@
 F 0 "TP6" V 4154 3388 50  0000 L CNN
 F 1 "4.43MHz" V 4245 3388 50  0000 L CNN
-F 2 "TestPoint:TestPoint_Pad_D1.5mm" H 4400 3200 50  0001 C CNN
+F 2 "TestPoint:TestPoint_THTPad_D2.0mm_Drill1.0mm" H 4400 3200 50  0001 C CNN
 F 3 "~" H 4400 3200 50  0001 C CNN
 	1    4200 3200
@@
 F 0 "TP3" H 758 3418 50  0000 L CNN
 F 1 "3.54MHz" H 758 3327 50  0000 L CNN
-F 2 "TestPoint:TestPoint_Pad_D1.5mm" H 900 3300 50  0001 C CNN
+F 2 "TestPoint:TestPoint_THTPad_D2.0mm_Drill1.0mm" H 900 3300 50  0001 C CNN
 F 3 "~" H 900 3300 50  0001 C CNN
 	1    700  3300
@@
 Connection ~ 10900 2350
 Connection ~ 11100 2350
+$Comp
+L Connector:TestPoint TP2
+U 1 1 61E63A0B
+P 5350 5450
+F 0 "TP2" H 5408 5568 50  0000 L CNN
+F 1 "A1_RES" H 5408 5477 50  0000 L CNN
+F 2 "TestPoint:TestPoint_THTPad_D2.0mm_Drill1.0mm" H 5550 5450 50  0001 C CNN
+F 3 "~" H 5550 5450 50  0001 C CNN
+	1    5350 5450
+	1    0    0    -1
+$EndComp
+Wire Wire Line
+	15250 4450 15250 4550
+Wire Wire Line
+	14750 5050 15650 5050
+Wire Wire Line
+	15650 4650 15400 4650
+Wire Wire Line
+	15400 4650 15400 4550
+Wire Wire Line
+	15400 4550 15250 4550
+Connection ~ 15250 4550
+Wire Wire Line
+	15250 4550 15250 4600
+Wire Wire Line
+	15650 4350 15900 4350
+Wire Wire Line
+	15900 4350 15900 4750
+Wire Wire Line
+	15900 4750 15650 4750
+Connection ~ 15650 4350
 Wire Bus Line
 	9900 9650 11550 9650
@@
 Wire Bus Line
 	11550 1750 11550 9650
-$Comp
-L Connector:TestPoint TP2
-U 1 1 61E63A0B
-P 5350 5450
-F 0 "TP2" H 5408 5568 50  0000 L CNN
-F 1 "A1_RES" H 5408 5477 50  0000 L CNN
-F 2 "TestPoint:TestPoint_Pad_D1.5mm" H 5550 5450 50  0001 C CNN
-F 3 "~" H 5550 5450 50  0001 C CNN
-	1    5350 5450
-	1    0    0    -1
-$EndComp
 $EndSCHEMATC
