File: OrigJrBoard/JrBoard/JrBoard.sch (KiCad schematic (older format))
At the start: 158 parts, among them J1 Joy left, J2 DC In, J3 Joy right, J4 RF_Out, J5 Cartridge Connector, J6 SEL / RES, Q1 2N3906, Q2 2N3906, Q3 2N3906, Q4 2N3904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

Commit message: Added Gerber files, going to production
Parts:
- added H1, H2, H4: MountingHole, Atari2600Jr:HoleEdge, symbol Mechanical:MountingHole
- added H3: MountingHole, Atari2600Jr:HoleTop, symbol Mechanical:MountingHole
Changed lines of the file:
@@
 Wire Bus Line
 	11550 1750 11550 9650
+$Comp
+L Mechanical:MountingHole H1
+U 1 1 6041EEB6
+P 600 11100
+F 0 "H1" H 700 11146 50  0000 L CNN
+F 1 "MountingHole" H 700 11055 50  0000 L CNN
+F 2 "Atari2600Jr:HoleEdge" H 600 11100 50  0001 C CNN
+F 3 "~" H 600 11100 50  0001 C CNN
+	1    600  11100
+	1    0    0    -1
+$EndComp
+$Comp
+L Mechanical:MountingHole H2
+U 1 1 6041F647
+P 600 10900
+F 0 "H2" H 700 10946 50  0000 L CNN
+F 1 "MountingHole" H 700 10855 50  0000 L CNN
+F 2 "Atari2600Jr:HoleEdge" H 600 10900 50  0001 C CNN
+F 3 "~" H 600 10900 50  0001 C CNN
+	1    600  10900
+	1    0    0    -1
+$EndComp
+$Comp
+L Mechanical:MountingHole H3
+U 1 1 6041F737
+P 600 10700
+F 0 "H3" H 700 10746 50  0000 L CNN
+F 1 "MountingHole" H 700 10655 50  0000 L CNN
+F 2 "Atari2600Jr:HoleTop" H 600 10700 50  0001 C CNN
+F 3 "~" H 600 10700 50  0001 C CNN
+	1    600  10700
+	1    0    0    -1
+$EndComp
+$Comp
+L Mechanical:MountingHole H4
+U 1 1 6041F9BA
+P 600 10500
+F 0 "H4" H 700 10546 50  0000 L CNN
+F 1 "MountingHole" H 700 10455 50  0000 L CNN
+F 2 "Atari2600Jr:HoleEdge" H 600 10500 50  0001 C CNN
+F 3 "~" H 600 10500 50  0001 C CNN
+	1    600  10500
+	1    0    0    -1
+$EndComp
 $EndSCHEMATC

Commit message: Minor corrections
Parts:
- C50: value 47n -> 47p
Changed lines of the file:
@@
 P 14100 8050
 F 0 "C50" H 14215 8096 50  0000 L CNN
-F 1 "47n" H 14215 8005 50  0000 L CNN
+F 1 "47p" H 14215 8005 50  0000 L CNN
 F 2 "Atari2600Jr:C_leg_small" H 14138 7900 50  0001 C CNN
 F 3 "~" H 14100 8050 50  0001 C CNN
@@
 	15900 4750 15650 4750
 Connection ~ 15650 4350
+$Comp
+L Mechanical:MountingHole H1
+U 1 1 6041EEB6
+P 600 11100
+F 0 "H1" H 700 11146 50  0000 L CNN
+F 1 "MountingHole" H 700 11055 50  0000 L CNN
+F 2 "Atari2600Jr:HoleEdge" H 600 11100 50  0001 C CNN
+F 3 "~" H 600 11100 50  0001 C CNN
+	1    600  11100
+	1    0    0    -1
+$EndComp
+$Comp
+L Mechanical:MountingHole H2
+U 1 1 6041F647
+P 600 10900
+F 0 "H2" H 700 10946 50  0000 L CNN
+F 1 "MountingHole" H 700 10855 50  0000 L CNN
+F 2 "Atari2600Jr:HoleEdge" H 600 10900 50  0001 C CNN
+F 3 "~" H 600 10900 50  0001 C CNN
+	1    600  10900
+	1    0    0    -1
+$EndComp
+$Comp
+L Mechanical:MountingHole H3
+U 1 1 6041F737
+P 600 10700
+F 0 "H3" H 700 10746 50  0000 L CNN
+F 1 "MountingHole" H 700 10655 50  0000 L CNN
+F 2 "Atari2600Jr:HoleTop" H 600 10700 50  0001 C CNN
+F 3 "~" H 600 10700 50  0001 C CNN
+	1    600  10700
+	1    0    0    -1
+$EndComp
+$Comp
+L Mechanical:MountingHole H4
+U 1 1 6041F9BA
+P 600 10500
+F 0 "H4" H 700 10546 50  0000 L CNN
+F 1 "MountingHole" H 700 10455 50  0000 L CNN
+F 2 "Atari2600Jr:HoleEdge" H 600 10500 50  0001 C CNN
+F 3 "~" H 600 10500 50  0001 C CNN
+	1    600  10500
+	1    0    0    -1
+$EndComp
 Wire Bus Line
 	9900 9650 11550 9650
@@
 Wire Bus Line
 	11550 1750 11550 9650
-$Comp
-L Mechanical:MountingHole H1
-U 1 1 6041EEB6
-P 600 11100
-F 0 "H1" H 700 11146 50  0000 L CNN
-F 1 "MountingHole" H 700 11055 50  0000 L CNN
-F 2 "Atari2600Jr:HoleEdge" H 600 11100 50  0001 C CNN
-F 3 "~" H 600 11100 50  0001 C CNN
-	1    600  11100
-	1    0    0    -1
-$EndComp
-$Comp
-L Mechanical:MountingHole H2
-U 1 1 6041F647
-P 600 10900
-F 0 "H2" H 700 10946 50  0000 L CNN
-F 1 "MountingHole" H 700 10855 50  0000 L CNN
-F 2 "Atari2600Jr:HoleEdge" H 600 10900 50  0001 C CNN
-F 3 "~" H 600 10900 50  0001 C CNN
-	1    600  10900
-	1    0    0    -1
-$EndComp
-$Comp
-L Mechanical:MountingHole H3
-U 1 1 6041F737
-P 600 10700
-F 0 "H3" H 700 10746 50  0000 L CNN
-F 1 "MountingHole" H 700 10655 50  0000 L CNN
-F 2 "Atari2600Jr:HoleTop" H 600 10700 50  0001 C CNN
-F 3 "~" H 600 10700 50  0001 C CNN
-	1    600  10700
-	1    0    0    -1
-$EndComp
-$Comp
-L Mechanical:MountingHole H4
-U 1 1 6041F9BA
-P 600 10500
-F 0 "H4" H 700 10546 50  0000 L CNN
-F 1 "MountingHole" H 700 10455 50  0000 L CNN
-F 2 "Atari2600Jr:HoleEdge" H 600 10500 50  0001 C CNN
-F 3 "~" H 600 10500 50  0001 C CNN
-	1    600  10500
-	1    0    0    -1
-$EndComp
 $EndSCHEMATC
