File: OrigJrBoard/JrBoard/JrBoard.kicad_pcb (KiCad board)
At the start: 2 copper layers, 247 x 132 mm, 162 parts, among them J1 Joy left, J2 DC In, J3 Joy right, J4 RF_Out, J5 Cartridge Connector, J6 SEL / RES, Q1 2N3906, Q2 2N3906, Q3 2N3906, Q4 2N3904, Q5 2N3904, T1 TV_Trans, Y1 3.546894MHz, Y2 4.433618MHz

Commit message: Minor corrections
Parts:
- C50: value 47n -> 47p
Changed lines of the file:
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@@
   )
   (setup
-    (last_trace_width 0.635)
+    (last_trace_width 0.25)
     (user_trace_width 0.127)
     (user_trace_width 0.635)
@@
   (module Atari2600Jr:Wire (layer F.Cu)
     (at 187.29 109.915)
-    (fp_text reference W3 (at -0.635 -1.27) (layer F.SilkS)
+    (fp_text reference W3 (at -3.175 -0.635) (layer F.SilkS)
       (effects (font (size 1 1) (thickness 0.15)))
     )
-    (fp_text value DNF (at 0 1.27) (layer F.Fab)
+    (fp_text value DNF (at 0 -0.635) (layer F.SilkS)
       (effects (font (size 1 1) (thickness 0.15)))
     )
@@
   (module Atari2600Jr:Wire (layer F.Cu)
     (at 121.25 142.3 270)
-    (fp_text reference W2 (at 0 -1.27 90) (layer F.SilkS)
+    (fp_text reference W2 (at 1.905 0.635 90) (layer F.SilkS)
       (effects (font (size 1 1) (thickness 0.15)))
     )
-    (fp_text value DNF (at 0 1.27 90) (layer F.Fab)
+    (fp_text value DNF (at -2.54 0.635 90) (layer F.SilkS)
       (effects (font (size 1 1) (thickness 0.15)))
     )
@@
   (module Atari2600Jr:Wire (layer F.Cu)
     (at 171.415 109.915)
-    (fp_text reference W1 (at 0 -1.27) (layer F.SilkS)
+    (fp_text reference W1 (at -2.54 -0.635) (layer F.SilkS)
       (effects (font (size 1 1) (thickness 0.15)))
     )
-    (fp_text value DNF (at 0 1.27) (layer F.Fab)
+    (fp_text value DNF (at 2.54 -0.635) (layer F.SilkS)
       (effects (font (size 1 1) (thickness 0.15)))
     )
@@
       (effects (font (size 1 1) (thickness 0.15)))
     )
-    (fp_text value DNF (at 0 0 90) (layer F.Fab)
+    (fp_text value DNF (at 0 0 90) (layer F.SilkS)
       (effects (font (size 1 1) (thickness 0.15)))
     )
@@
       (effects (font (size 1 1) (thickness 0.15)))
     )
-    (fp_text value DNF (at 0 0 90) (layer F.Fab)
+    (fp_text value DNF (at 0 0 90) (layer F.SilkS)
       (effects (font (size 1 1) (thickness 0.15)))
     )
@@
       (effects (font (size 1 1) (thickness 0.15)))
     )
-    (fp_text value 47n (at 0 0 90) (layer F.SilkS)
+    (fp_text value 47p (at 0 0 90) (layer F.SilkS)
       (effects (font (size 1 1) (thickness 0.15)))
     )
@@
       (effects (font (size 1 1) (thickness 0.15)))
     )
-    (fp_text value DNF (at 0 0 90) (layer F.Fab)
+    (fp_text value DNF (at 0 0 90) (layer F.SilkS)
       (effects (font (size 1 1) (thickness 0.15)))
     )
@@
   (gr_line (start 106 23) (end 193 23) (layer Edge.Cuts) (width 0.05))
   (gr_line (start 26 40) (end 26 124) (layer Edge.Cuts) (width 0.05))
-  (segment (start 211 39.6) (end 211.8 38.8) (width 0.127) (layer F.Cu) (net 40))
-  (segment (start 211.8 38.8) (end 212.4 38.2) (width 0.127) (layer F.Cu) (net 40))
-  (segment (start 212.4 38.2) (end 213.8 39.6) (width 0.127) (layer F.Cu) (net 40))
-  (segment (start 213.8 39.6) (end 215.2 38.2) (width 0.127) (layer F.Cu) (net 40))
-  (segment (start 215.2 38.2) (end 216.6 39.6) (width 0.127) (layer F.Cu) (net 40))
-  (segment (start 216.6 39.6) (end 218 38.2) (width 0.127) (layer F.Cu) (net 40))
-  (segment (start 218 38.2) (end 219.4 39.6) (width 0.127) (layer F.Cu) (net 40))
-  (segment (start 219.4 39.6) (end 220.8 38.2) (width 0.127) (layer F.Cu) (net 40))
-  (segment (start 220.8 38.2) (end 222.2 39.6) (width 0.127) (layer F.Cu) (net 40))
-  (segment (start 222.2 39.6) (end 222.2 41.3) (width 0.127) (layer F.Cu) (net 40))
-  (segment (start 219.4 39.6) (end 219.4 41.3) (width 0.127) (layer F.Cu) (net 40))
-  (segment (start 216.6 39.6) (end 216.6 41.3) (width 0.127) (layer F.Cu) (net 40))
-  (segment (start 211 39.6) (end 210.9 39.5) (width 0.127) (layer F.Cu) (net 40))
-  (segment (start 210.9 39.5) (end 210.893501 39.493501) (width 0.127) (layer F.Cu) (net 40))
-  (segment (start 210.893501 39.493501) (end 209.9 38.5) (width 0.127) (layer F.Cu) (net 40))
-  (segment (start 209.9 38.5) (end 209.6 38.2) (width 0.127) (layer F.Cu) (net 40))
-  (segment (start 209.6 38.2) (end 208.2 39.6) (width 0.127) (layer F.Cu) (net 40))
-  (segment (start 208.2 39.6) (end 208.1 39.7) (width 0.127) (layer F.Cu) (net 40))
-  (segment (start 208.1 39.7) (end 208.1 41.3) (width 0.127) (layer F.Cu) (net 40))
-  (segment (start 211 39.6) (end 211 41.6) (width 0.127) (layer F.Cu) (net 40))
-  (segment (start 213.8 39.6) (end 213.8 41.3) (width 0.127) (layer F.Cu) (net 40))
-  (segment (start 220.8 38.2) (end 220.8 36.2) (width 0.127) (layer F.Cu) (net 40))
-  (segment (start 220.8 36.2) (end 218 36.2) (width 0.127) (layer F.Cu) (net 40))
-  (segment (start 218 36.2) (end 218 38.2) (width 0.127) (layer F.Cu) (net 40))
-  (segment (start 218 36.2) (end 215.2 36.2) (width 0.127) (layer F.Cu) (net 40))
-  (segment (start 215.2 36.2) (end 215.2 38.2) (width 0.127) (layer F.Cu) (net 40))
   (segment (start 132.045 102.295) (end 132.045 89.595) (width 0.25) (layer F.Cu) (net 1))
   (segment (start 132.045 111.185) (end 132.045 108.01) (width 0.25) (layer F.Cu) (net 1))
@@
   (segment (start 93.31 80.07) (end 95.215 81.975) (width 0.635) (layer B.Cu) (net 39))
   (segment (start 95.215 81.975) (end 127.6 81.975) (width 0.635) (layer B.Cu) (net 39))
+  (segment (start 211 39.6) (end 211.8 38.8) (width 0.127) (layer F.Cu) (net 40))
+  (segment (start 211.8 38.8) (end 212.4 38.2) (width 0.127) (layer F.Cu) (net 40))
+  (segment (start 212.4 38.2) (end 213.8 39.6) (width 0.127) (layer F.Cu) (net 40))
+  (segment (start 213.8 39.6) (end 215.2 38.2) (width 0.127) (layer F.Cu) (net 40))
+  (segment (start 215.2 38.2) (end 216.6 39.6) (width 0.127) (layer F.Cu) (net 40))
+  (segment (start 216.6 39.6) (end 218 38.2) (width 0.127) (layer F.Cu) (net 40))
+  (segment (start 218 38.2) (end 219.4 39.6) (width 0.127) (layer F.Cu) (net 40))
+  (segment (start 219.4 39.6) (end 220.8 38.2) (width 0.127) (layer F.Cu) (net 40))
+  (segment (start 220.8 38.2) (end 222.2 39.6) (width 0.127) (layer F.Cu) (net 40))
+  (segment (start 222.2 39.6) (end 222.2 41.3) (width 0.127) (layer F.Cu) (net 40))
+  (segment (start 219.4 39.6) (end 219.4 41.3) (width 0.127) (layer F.Cu) (net 40))
+  (segment (start 216.6 39.6) (end 216.6 41.3) (width 0.127) (layer F.Cu) (net 40))
+  (segment (start 211 39.6) (end 210.9 39.5) (width 0.127) (layer F.Cu) (net 40))
+  (segment (start 210.9 39.5) (end 210.893501 39.493501) (width 0.127) (layer F.Cu) (net 40))
+  (segment (start 210.893501 39.493501) (end 209.9 38.5) (width 0.127) (layer F.Cu) (net 40))
+  (segment (start 209.9 38.5) (end 209.6 38.2) (width 0.127) (layer F.Cu) (net 40))
+  (segment (start 209.6 38.2) (end 208.2 39.6) (width 0.127) (layer F.Cu) (net 40))
+  (segment (start 208.2 39.6) (end 208.1 39.7) (width 0.127) (layer F.Cu) (net 40))
+  (segment (start 208.1 39.7) (end 208.1 41.3) (width 0.127) (layer F.Cu) (net 40))
+  (segment (start 211 39.6) (end 211 41.6) (width 0.127) (layer F.Cu) (net 40))
+  (segment (start 213.8 39.6) (end 213.8 41.3) (width 0.127) (layer F.Cu) (net 40))
+  (segment (start 220.8 38.2) (end 220.8 36.2) (width 0.127) (layer F.Cu) (net 40))
+  (segment (start 220.8 36.2) (end 218 36.2) (width 0.127) (layer F.Cu) (net 40))
+  (segment (start 218 36.2) (end 218 38.2) (width 0.127) (layer F.Cu) (net 40))
+  (segment (start 218 36.2) (end 215.2 36.2) (width 0.127) (layer F.Cu) (net 40))
+  (segment (start 215.2 36.2) (end 215.2 38.2) (width 0.127) (layer F.Cu) (net 40))
   (segment (start 230.717501 134.432499) (end 230.857499 134.432499) (width 0.635) (layer B.Cu) (net 40))
   (segment (start 230.717501 134.432499) (end 229.741599 134.432499) (width 0.635) (layer B.Cu) (net 40))
