File: ModdedJrBoard/JrBoard.sch (KiCad schematic (older format))
At the start: 148 parts, among them J1 Joy left, J2 DC In, J3 Joy right, J4 A/V, J5 Cartridge Connector, J6 SEL / RES, Q1 2N3906, Q2 2N3906, Q5 2N3904, Q6 2N3906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

Commit message: Schematic corrections
Parts:
- A6: footprint (none) -> Package_DIP:DIP-8_W7.62mm
- A7: footprint (none) -> Package_DIP:DIP-14_W7.62mm
Changed lines of the file:
@@
 Connection ~ 13800 9100
 $Comp
-L power:GND #PWR?
+L power:GND #PWR0124
 U 1 1 6015F0E8
 P 13800 9400
-F 0 "#PWR?" H 13800 9150 50  0001 C CNN
+F 0 "#PWR0124" H 13800 9150 50  0001 C CNN
 F 1 "GND" H 13805 9227 50  0000 C CNN
 F 2 "" H 13800 9400 50  0001 C CNN
@@
 $EndComp
 $Comp
-L power:GND #PWR?
+L power:GND #PWR0125
 U 1 1 602E2BA2
 P 15100 7250
-F 0 "#PWR?" H 15100 7000 50  0001 C CNN
+F 0 "#PWR0125" H 15100 7000 50  0001 C CNN
 F 1 "GND" H 15105 7077 50  0000 C CNN
 F 2 "" H 15100 7250 50  0001 C CNN
@@
 $EndComp
 $Comp
-L power:+5V #PWR?
+L power:+5V #PWR0135
 U 1 1 607693AA
 P 14400 4800
-F 0 "#PWR?" H 14400 4650 50  0001 C CNN
+F 0 "#PWR0135" H 14400 4650 50  0001 C CNN
 F 1 "+5V" V 14415 4928 50  0000 L CNN
 F 2 "" H 14400 4800 50  0001 C CNN
@@
 F 0 "A6" H 13000 5700 50  0000 C CNN
 F 1 "NE555" H 13050 5600 50  0000 C CNN
-F 2 "" H 12850 5200 50  0001 C CNN
+F 2 "Package_DIP:DIP-8_W7.62mm" H 12850 5200 50  0001 C CNN
 F 3 "http://www.ti.com/lit/ds/symlink/ne555.pdf" H 12850 5200 50  0001 C CNN
 	1    12850 5200
@@
 $EndComp
 $Comp
-L power:GND #PWR?
+L power:GND #PWR0153
 U 1 1 607B9D9E
 P 12850 5600
-F 0 "#PWR?" H 12850 5350 50  0001 C CNN
+F 0 "#PWR0153" H 12850 5350 50  0001 C CNN
 F 1 "GND" H 12855 5427 50  0000 C CNN
 F 2 "" H 12850 5600 50  0001 C CNN
@@
 $EndComp
 $Comp
-L power:GND #PWR?
+L power:GND #PWR0165
 U 1 1 607BA8FA
 P 11900 5750
-F 0 "#PWR?" H 11900 5500 50  0001 C CNN
+F 0 "#PWR0165" H 11900 5500 50  0001 C CNN
 F 1 "GND" H 11905 5577 50  0000 C CNN
 F 2 "" H 11900 5750 50  0001 C CNN
@@
 $EndComp
 $Comp
-L power:+5V #PWR?
+L power:+5V #PWR0166
 U 1 1 608097D6
 P 12850 4600
-F 0 "#PWR?" H 12850 4450 50  0001 C CNN
+F 0 "#PWR0166" H 12850 4450 50  0001 C CNN
 F 1 "+5V" V 12865 4728 50  0000 L CNN
 F 2 "" H 12850 4600 50  0001 C CNN
@@
 $EndComp
 $Comp
-L power:GND #PWR?
+L power:GND #PWR0167
 U 1 1 60E50797
 P 13600 5850
-F 0 "#PWR?" H 13600 5600 50  0001 C CNN
+F 0 "#PWR0167" H 13600 5600 50  0001 C CNN
 F 1 "GND" H 13605 5677 50  0000 C CNN
 F 2 "" H 13600 5850 50  0001 C CNN
@@
 $EndComp
 $Comp
-L power:GND #PWR?
+L power:GND #PWR0168
 U 1 1 610896C3
 P 8000 1600
-F 0 "#PWR?" H 8000 1350 50  0001 C CNN
+F 0 "#PWR0168" H 8000 1350 50  0001 C CNN
 F 1 "GND" H 8005 1427 50  0000 C CNN
 F 2 "" H 8000 1600 50  0001 C CNN
@@
 F 0 "A7" H 6130 4146 50  0000 L CNN
 F 1 "74LS00" H 6130 4055 50  0000 L CNN
-F 2 "" H 5900 4100 50  0001 C CNN
+F 2 "Package_DIP:DIP-14_W7.62mm" H 5900 4100 50  0001 C CNN
 F 3 "http://www.ti.com/lit/gpn/sn74ls00" H 5900 4100 50  0001 C CNN
 	5    5900 4100
@@
 $EndComp
 $Comp
-L power:GND #PWR?
+L power:GND #PWR0169
 U 1 1 6128E5E8
 P 5900 4600
-F 0 "#PWR?" H 5900 4350 50  0001 C CNN
+F 0 "#PWR0169" H 5900 4350 50  0001 C CNN
 F 1 "GND" H 5905 4427 50  0000 C CNN
 F 2 "" H 5900 4600 50  0001 C CNN
@@
 $EndComp
 $Comp
-L power:GND #PWR?
+L power:GND #PWR0170
 U 1 1 6128FB4B
 P 6100 3550
-F 0 "#PWR?" H 6100 3300 50  0001 C CNN
+F 0 "#PWR0170" H 6100 3300 50  0001 C CNN
 F 1 "GND" H 6105 3377 50  0000 C CNN
 F 2 "" H 6100 3550 50  0001 C CNN
@@
 F 0 "A7" H 7650 2725 50  0000 C CNN
 F 1 "74LS00" H 7650 2634 50  0000 C CNN
-F 2 "" H 7650 2400 50  0001 C CNN
+F 2 "Package_DIP:DIP-14_W7.62mm" H 7650 2400 50  0001 C CNN
 F 3 "http://www.ti.com/lit/gpn/sn74ls00" H 7650 2400 50  0001 C CNN
 	1    7650 2400
@@
 F 0 "A7" H 7650 3325 50  0000 C CNN
 F 1 "74LS00" H 7650 3234 50  0000 C CNN
-F 2 "" H 7650 3000 50  0001 C CNN
+F 2 "Package_DIP:DIP-14_W7.62mm" H 7650 3000 50  0001 C CNN
 F 3 "http://www.ti.com/lit/gpn/sn74ls00" H 7650 3000 50  0001 C CNN
 	2    7650 3000
@@
 F 0 "A7" H 7650 3975 50  0000 C CNN
 F 1 "74LS00" H 7650 3884 50  0000 C CNN
-F 2 "" H 7650 3650 50  0001 C CNN
+F 2 "Package_DIP:DIP-14_W7.62mm" H 7650 3650 50  0001 C CNN
 F 3 "http://www.ti.com/lit/gpn/sn74ls00" H 7650 3650 50  0001 C CNN
 	3    7650 3650
@@
 F 0 "A7" H 7650 4575 50  0000 C CNN
 F 1 "74LS00" H 7650 4484 50  0000 C CNN
-F 2 "" H 7650 4250 50  0001 C CNN
+F 2 "Package_DIP:DIP-14_W7.62mm" H 7650 4250 50  0001 C CNN
 F 3 "http://www.ti.com/lit/gpn/sn74ls00" H 7650 4250 50  0001 C CNN
 	4    7650 4250
@@
 Connection ~ 8850 3250
 $Comp
-L power:GND #PWR?
+L power:GND #PWR0171
 U 1 1 619D3F8F
 P 8850 3550
-F 0 "#PWR?" H 8850 3300 50  0001 C CNN
+F 0 "#PWR0171" H 8850 3300 50  0001 C CNN
 F 1 "GND" H 8855 3377 50  0000 C CNN
 F 2 "" H 8850 3550 50  0001 C CNN
@@
 Wire Wire Line
 	8450 3000 8450 2000
-Wire Bus Line
-	9900 9650 11550 9650
-Wire Bus Line
-	3150 7150 3150 9650
-Wire Bus Line
-	9900 6600 9900 9650
-Wire Bus Line
-	2100 6950 2100 9650
-Wire Bus Line
-	8050 6850 8050 9650
-Wire Bus Line
-	6700 6850 6700 9650
-Wire Bus Line
-	5550 6600 5550 9650
-Wire Bus Line
-	3850 6600 3850 9650
-Wire Bus Line
-	11550 1750 11550 9650
 Wire Wire Line
 	8450 3000 8400 3000
@@
 Wire Wire Line
 	8850 2000 8850 3250
+Wire Bus Line
+	9900 9650 11550 9650
+Wire Bus Line
+	3150 7150 3150 9650
+Wire Bus Line
+	9900 6600 9900 9650
+Wire Bus Line
+	2100 6950 2100 9650
+Wire Bus Line
+	8050 6850 8050 9650
+Wire Bus Line
+	6700 6850 6700 9650
+Wire Bus Line
+	5550 6600 5550 9650
+Wire Bus Line
+	3850 6600 3850 9650
+Wire Bus Line
+	11550 1750 11550 9650
 $EndSCHEMATC

Commit message: Right footprints for diode
Parts:
- D70, D71: footprint Diode_THT:D_DO-35_SOD27_P7.62mm_Horizontal -> Atari2600Jr:Diode
Changed lines of the file:
@@
 F 0 "D70" H 8250 2784 50  0000 C CNN
 F 1 "1N4148" H 8250 2875 50  0000 C CNN
-F 2 "Diode_THT:D_DO-35_SOD27_P7.62mm_Horizontal" H 8250 2825 50  0001 C CNN
+F 2 "Atari2600Jr:Diode" H 8250 2825 50  0001 C CNN
 F 3 "https://assets.nexperia.com/documents/data-sheet/1N4148_1N4448.pdf" H 8250 3000 50  0001 C CNN
 	1    8250 3000
@@
 F 0 "D71" H 8600 3034 50  0000 C CNN
 F 1 "1N4148" H 8600 3125 50  0000 C CNN
-F 2 "Diode_THT:D_DO-35_SOD27_P7.62mm_Horizontal" H 8600 3075 50  0001 C CNN
+F 2 "Atari2600Jr:Diode" H 8600 3075 50  0001 C CNN
 F 3 "https://assets.nexperia.com/documents/data-sheet/1N4148_1N4448.pdf" H 8600 3250 50  0001 C CNN
 	1    8600 3250
